File: pcb/thpdl_2511.kicad_pcb (KiCad board)
At the start: 2 copper layers, 82.4 x 46 mm, 36 parts

Commit message: add pcb version to silkscreen and add 3d redner pic to readme
Other:
- board text added: "Development Board V1.0 Stratos Thivaios (C) 2025 https://github.com/sthivaios"
- board text removed: "Development Board Stratos Thivaios (C) 2025 https://github.com/sthivaios"
Changed lines of the file:
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@@
 		(layer "Edge.Cuts")
 	)
-	(gr_text "\nDevelopment Board\nStratos Thivaios (C) 2025\nhttps://github.com/sthivaios"
+	(gr_text "\nDevelopment Board V1.0\nStratos Thivaios (C) 2025\nhttps://github.com/sthivaios"
 		(at 136.2 114.6 0)
 		(layer "F.SilkS")
