File: pcb/thpdl_2511.kicad_pcb (KiCad board)
At the start: 2 copper layers, 82.4 x 46 mm, 36 parts

Commit message: add i2c header
Parts:
- added I2C1: Conn_01x03_Pin, Connector_PinHeader_2.54mm:PinHeader_1x03_P2.54mm_Vertical, F.Cu at (173.5, 110.0)
Routing:
- net SDA: track 34.2 -> 52.8 mm, vias 2 -> 4
- net SCL: track 36.0 -> 51.6 mm
